File: CAD_resources/test1.brd (EAGLE design)
At the start: 147.3 x 157.2 mm, 83 parts, among them J2 230V, J3 J1B1211CCD, Q1 BSS84, Q2 29MHz, Q5 32.768, T1 3FD-312, U1 STM32F103C8T6LQFP48_STM-M, U2 LM2576-3.3WTTO-220-5_LB03(B8X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, U3 LM2940CT-5.0/NOPBT03B, U4 W550048LQFP_W5500_WIZ-M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

Commit message: added gebber files
Parts:
- U2: value LM2576-3.3WTTO-220-5_LB03(B8X)_MCH -> LM2576-3.3WT; device regu3:TO-220-5_LB03(B8X)_MCH -> LM2576-3.3WT:TO170P1054X470X1514-5
- moved C4 269.1 mm to (-129.5, 1.27)
- moved D4 261.9 mm to (-110.5, 116.8), flipped to the bottom
- moved D3 254.1 mm to (-96.5, 95.2)
- moved LED1 249.3 mm to (-120.7, 78.7)
- moved C25 247.2 mm to (-96.5, 105.4)
- moved C18 246.5 mm to (-116.8, 139.7)
- moved D2 245.4 mm to (-83.8, 78.7)
- moved C21 241.1 mm to (-121.9, 118.1), flipped to the bottom
- moved L1 235.7 mm to (-99.1, 74.9), flipped to the top
- moved R5 230.8 mm to (-69.8, 132.1)
- moved J2 230.1 mm to (-30.5, 95.2), turned to 0 degrees
- moved U1 229.0 mm to (-108.0, 35.6), turned to 0 degrees
- moved R7 226.6 mm to (-82.5, 125.7)
- moved R17 225.4 mm to (-108.0, 130.8)
- moved LED2 222.8 mm to (-114.3, 17.8)
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Connections:
- new net N$35: C2.1, U2.1
- net GND: now also C2.2; no longer C2.1
- net VIN: no longer C2.2, U2.1
Routing:
- net GND: track 0.00 -> 1114.4 mm, vias 0 -> 1
- net V3.3: track 0.00 -> 573.0 mm, vias 0 -> 13
- net V3.3A: track 0.00 -> 512.8 mm, vias 0 -> 6
- net N$10: track 0.00 -> 322.2 mm, vias 0 -> 1
- net N$22: track 0.00 -> 261.2 mm, vias 0 -> 4
- net N$24: track 0.00 -> 250.8 mm, vias 0 -> 5
- net VIN: track 0.00 -> 242.9 mm, vias 0 -> 2
- net BUSL1: track 0.00 -> 234.0 mm, vias 0 -> 1
- net BUSL2: track 0.00 -> 232.4 mm
- net N$51: track 0.00 -> 216.4 mm, vias 0 -> 2
- net LED3: track 0.00 -> 207.7 mm, vias 0 -> 1
- net N$11: track 0.00 -> 185.9 mm, vias 0 -> 2
- net N$27: track 0.00 -> 170.4 mm, vias 0 -> 4
- net N$31: track 0.00 -> 167.4 mm, vias 0 -> 4
- net SCSN: track 0.00 -> 163.1 mm, vias 0 -> 1
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Other:
- board size 147.3 x 157.2 mm -> 181.6 x 176.2 mm
