File: CAD_resources/watCals_schmatic.sch (EAGLE design)
At the start: 75 parts, among them J3 J1B1211CCD, Q1 BSS84, Q2 29MHz, Q5 32.768, U1 STM32F103C8T6LQFP48_STM-M, U2 LM2576-3.3WTTO-220-5_LB03(B8X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, U3 LM2940CT-5.0/NOPBT03B, U4 W550048LQFP_W5500_WIZ-M, U5 TSS721ADD16_TEX

Commit message: added gebber
Parts:
- removed J1: (no value), con-jack:DCJ0303
- added C32: 470uF, rcl:CPOL-EUE2,5-6E
- added C33: 1u, capacitor-wima:C2.5/2
- added D1, D3, D4, D5: 1N4004, diode:1N4004
- added G1: CR2032V, battery:CR2032V
- added J2: 230V, con-amp:MTA02-100
- added T1: 3FD-312, 3FD-312:3FD-312
- C6: value (none) -> 300
- C7, C8, C9: value (none) -> 0.1u
- U2: value LM2576-3.3WTTO-220-5_LB03(B8X)_MCH -> LM2576-3.3WT; device regu3:LM2576-3.3WTTO-220-5_LB03(B8X)_MCH -> LM2576-3.3WT:LM2576-3.3WT
Connections:
- removed net N$36: SV1.4
- removed net N$37: SV1.2
- removed net N$38: SV1.9
- removed net PB10: LED3.A, U1A.PB10
- removed net PB8: LED2.A, U1A.PB8
- removed net PB9: LED1.A, U1A.PB9
- new net LED1: LED1.A, U1A.PA8
- new net LED2: LED2.A, U1A.PA9
- new net LED3: LED3.A, U1A.PA10
- new net N$41: T1.6, T1.7
- new net N$44: J2.2, T1.1
- new net N$45: T1.2, T1.3
- new net N$47: J2.1, T1.4
- new net N$48: D1.C, D5.A, T1.5
- new net N$51: D3.C, D4.A, T1.8
- new net RXI: U1A.PB11, U5.RXI
- net GND: now also C2.2, C32.-, C33.2, D1.A, D3.A, U1B.VSSA, U2.!ON!/OFF, U2.GND; no longer C2.1, U2.!ON/OFF, U2.GROUND
- net JTCK: now also SV1.4; no longer SV1.7
- net JTDO: now also SV1.2; no longer SV1.3
- net JTMS: now also SV1.3; no longer SV1.5
- net N$10: now also R4.2
- net N$33: now also G1.+, U1B.VBAT; no longer SV1.10
- net N$34: now also C33.1, G1.-; no longer SV1.8
- net N$35: now also C2.1, U2.VIN; no longer SV1.6
- net N$9: no longer R4.1
- net PMODE0: now also U1A.PB0
- net PMODE1: now also U1A.PB1
- net PMODE2: now also U1A.PB2
- net V3.3: now also U1B.VDDA
- net V3.3A: now also R4.1; no longer R4.2
- net VIN: now also C32.+, D4.C, D5.C; no longer C2.2, U2.VIN

Commit message: added meters
Parts:
- C26: value 0.1u -> 0.1uF
- C27: value 10u -> 10u/16v
- L1: value (none) -> 100uH
- L2: value (none) -> 120 %5/50mA
- LED1: value (none) -> RED
- LED2: value (none) -> BLUE
- LED3: value (none) -> GREEN
- Q4: value (none) -> 8MHz
- R5, R6, R7: value (none) -> 1K
Connections:
- removed net N$19 (its old number): U4.SCSN
- removed net PF: U5.PF
- removed net SCSN: R15.2, R16.2, U1A.PA0-WKUP, U4.XO
- new net N$36: R15.2, R16.2, U4.XO
- new net SCS: U1A.PA0-WKUP, U4.SCSN
Other:
- moved on the sheet: R16
